File: KiCad/Practice/Practice.kicad_pcb (KiCad board)
At the start: 2 copper layers, 110 x 70 mm, 30 parts

Commit message: Development
Parts:
- removed the REF** at (119.4, 82.0)
- removed the REF** at (118.8, 100.6)
- removed TOP: LayerMarker_2_3.81x2.54mm_TextH1mm_P1.27mm_Named, Symbol:LayerMarker_2_3.81x2.54mm_TextH1mm_P1.27mm_Named
- added C3: 100n, Capacitor_THT:C_Disc_D7.5mm_W2.5mm_P5.00mm, F.Cu at (103.6, 117.5)
- added G***: LOGO, Lomis Company Logos:LomisCo1800s-20mm, F.Cu at (197.0, 118.0)
- added G***: LOGO, Virginia Tech Logos:VirginiaTech-Vert-20mm, F.Cu at (126.0, 85.0)
- added R10: 10k, Resistor_THT:R_Axial_DIN0207_L6.3mm_D2.5mm_P7.62mm_Horizontal, F.Cu at (171.2, 85.0)
- added R11: 1.2k, Resistor_THT:R_Axial_DIN0207_L6.3mm_D2.5mm_P7.62mm_Horizontal, F.Cu at (181.0, 124.1)
- added REF**: KiCad-Logo2_5mm_SilkScreen, Symbol:KiCad-Logo2_5mm_SilkScreen, F.Cu at (109.0, 80.0)
- added REF**: LayerMarker_2_3.81x2.54mm_TextH1mm_P1.27mm_Named_BottomMirr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, Symbol:LayerMarker_2_3.81x2.54mm_TextH1mm_P1.27mm_Named_BottomMirrored, F.Cu at (120.0, 128.0)
- added REF**: OSHW-Logo2_9.8x8mm_SilkScreen, Symbol:OSHW-Logo2_9.8x8mm_SilkScreen, F.Cu at (107.0, 88.0)
- J1: renamed from Power Input
- RN1: renamed from Resistor Network
- SW1: renamed from Input Switches
- SW2: renamed from Clock Enable
- U1: renamed from 74HC273; value 74HC273 -> 74AHC273
- renumbered 555-Timer to U2
Connections:
- SW2 pad 1: Net-(U2-Q) -> Net-(R11-Pad1)
Routing:
- net (no net): track 23.9 -> 0.00 mm
- net Net-(R11-Pad1): track 0.00 -> 12.0 mm
- net Net-(U1-Cp): track 29.7 -> 37.3 mm
- net +5V: track 121.5 -> 127.9 mm
- net Net-(U2-Q): track 33.5 -> 30.4 mm
Other:
- board text added: "11/19/2025 - v1.1 - Virginia Tech AMP Lab - Whittemore Hall"
- board text removed: "9/20/2025 - v1.0 - Virginia Tech AMP Lab - Whittemore Hall"

Commit message: Development updates to the LED Demo D-Type Flip Flop Board
Parts:
- added D9: 1N4001, Diode_THT:D_DO-41_SOD81_P10.16mm_Horizontal, F.Cu at (130.2, 122.0)
- added G***: LOGO, Virginia Tech Logos:AMP Lab, F.Cu at (195.8, 83.2)
- J1: value Conn_01x02_Pin -> Barrel_Jack_MountingPin; footprint Connector_PinHeader_2.54mm:PinHeader_1x02_P2.54mm_Vertical -> Connector_BarrelJack:BarrelJack_CUI_PJ-063AH_Horizontal
- moved C3 26.7 mm to (130.2, 115.8), turned to 180 degrees
- moved J1 9.09 mm to (112.5, 122.0), turned to -90 degrees
- moved REF** 7.00 mm to (127.0, 128.0)
- moved G*** 6.35 mm to (119.0, 94.0)
Connections:
- J1 pad 1: +5V -> Net-(D9-A)
Routing:
- net +5V: track 127.9 -> 97.9 mm
- net Net-(D9-A): track 0.00 -> 7.50 mm
Other:
- copper layers 2 -> 4
- rule solder_mask_min_width: 0.1016 -> 0.12
- board text added: "0.68k Resistor Network"
- board text added: "01/31/2026 - v1.2 - Virginia Tech AMP Lab - Whittemore Hall"
- board text added: "1.2k"
- board text added: "1N4k1"
- board text added: "555 Timer"
- board text added: "74AHC273"
- board text added: "JLCJLCJLCJLC"
- board text removed: "11/19/2025 - v1.1 - Virginia Tech AMP Lab - Whittemore Hall"
